File: Le_kube/Le_kube.sch (KiCad schematic (older format))
At the start: 12 parts

Commit message: sheet finish ?
Parts:
- added C1: 100nF, symbol Kube_library:C
- added C2: 10µF, symbol Kube_library:C
- added C3: 0.1µF, symbol Device:C_Small
- added C4, C5: 34pF, symbol Device:C_Small
- added C6: 10µF, symbol Device:C_Small
- added J?: USB_A, symbol Connector:USB_A
- added Q?: IRLB8721PBF, Package_TO_SOT_THT:TO-220-3_Vertical, symbol Transistor_FET:IRLB8721PBF
- added R15: 10K, symbol Kube_library:R
- added SW1: I/O, symbol Switch:SW_SPST
- added VR1: LD1117, symbol Kube_library:LD1117
- added Y?: Crystal, symbol Kube_library:Crystal
- R2: renamed from R?; value R_Small -> 10K
- R3, R4, R5: renamed from R?; value R_Small -> 220R
- SW2: renamed from SW?; value SW_Push -> RST
- gave numbers to parts that had none: 1
Connections:
- net labels added: +5V, ESP_RX, ESP_TX, HUM, ISP_MISO, ISP_MOSI, ISP_SCK, SCL, SCREEN_MISO, SCREEN_MOSI, SCREEN_RST, SCREEN_SCK, SCREEN_SS, SDA
- wire segments 42 -> 87
- no-connect marks 3 -> 9
Other:
- moved on the sheet: R1, R2, R3, R4, R5, U?

Commit message: fin de la schematic
Parts:
- added C18: 100nF, symbol Device:C_Small
- added CP0: 10µF, symbol Device:CP
- C6: value 10µF -> 100nF
- R3, R4, R5: value 220R -> 10K
- gave numbers to parts that had none: 9
- renumbered R15 to R16
Connections:
- wire segments 87 -> 98
- no-connect marks 9 -> 12
Other:
- moved on the sheet: SW1

Commit message: connector jack DC add
Parts:
- added J3: Jack-DC, symbol Connector:Jack-DC
- C1, C2: symbol Kube_library:C -> Le_kube-rescue:C-Kube_library
Connections:
- wire segments 98 -> 100
Changed lines of the file:
@@
 	2700 1100 2700 900
 $Comp
-L Kube_library:C C2
+L Le_kube-rescue:C-Kube_library C2
 U 1 1 60904FF9
 P 2700 1250
@@
 	1900 1400 2300 1400
 $Comp
-L Kube_library:C C1
+L Le_kube-rescue:C-Kube_library C1
 U 1 1 609039B3
 P 1900 1250
@@
 $EndComp
 $Comp
-L power:+5V #PWR?
+L power:+5V #PWR0114
 U 1 1 60DDA66B
-P 1050 900
-F 0 "#PWR?" H 1050 750 50  0001 C CNN
-F 1 "+5V" H 1065 1073 50  0000 C CNN
-F 2 "" H 1050 900 50  0001 C CNN
-F 3 "" H 1050 900 50  0001 C CNN
-	1    1050 900
-	0    -1   -1   0
-$EndComp
+P 1200 1350
+F 0 "#PWR0114" H 1200 1200 50  0001 C CNN
+F 1 "+5V" H 1215 1523 50  0000 C CNN
+F 2 "" H 1200 1350 50  0001 C CNN
+F 3 "" H 1200 1350 50  0001 C CNN
+	1    1200 1350
+	-1   0    0    1
+$EndComp
+$Comp
+L Connector:Jack-DC J?
+U 1 1 607A5C33
+P 750 1000
+AR Path="/608A4ECC/607A5C33" Ref="J?"  Part="1"
+AR Path="/607A5C33" Ref="J3"  Part="1"
+F 0 "J3" H 521 958 50  0000 R CNN
+F 1 "Jack-DC" H 521 1049 50  0000 R CNN
+F 2 "" H 800 960 50  0001 C CNN
+F 3 "~" H 800 960 50  0001 C CNN
+	1    750  1000
+	1    0    0    1
+$EndComp
+Wire Wire Line
+	1050 1100 1200 1100
+Wire Wire Line
+	1200 1100 1200 1350
 $EndSCHEMATC

Commit message: corrections
Parts:
- renumbered R16 to R15
Changed lines of the file:
@@
-$EndComp
-$Comp
-L Kube_library:R R16
-U 1 1 6095BC8F
-P 2700 5100
-F 0 "R16" H 2700 5325 50  0000 C CNN
-F 1 "10K" H 2700 5234 50  0000 C CNN
-F 2 "" H 2700 5100 50  0001 C CNN
-F 3 "" H 2700 5100 50  0001 C CNN
-	1    2700 5100
-	0    -1   -1   0
 $EndComp
 $Comp
@@
 	0    1    1    0
 $EndComp
-Connection ~ 2700 4900
 Wire Wire Line
 	2700 2350 2700 4900
@@
 L power:+5V #PWR0114
 U 1 1 60DDA66B
-P 1200 1350
-F 0 "#PWR0114" H 1200 1200 50  0001 C CNN
-F 1 "+5V" H 1215 1523 50  0000 C CNN
-F 2 "" H 1200 1350 50  0001 C CNN
-F 3 "" H 1200 1350 50  0001 C CNN
-	1    1200 1350
-	-1   0    0    1
+P 1050 900
+F 0 "#PWR0114" H 1050 750 50  0001 C CNN
+F 1 "+5V" H 1065 1073 50  0000 C CNN
+F 2 "" H 1050 900 50  0001 C CNN
+F 3 "" H 1050 900 50  0001 C CNN
+	1    1050 900
+	0    -1   -1   0
 $EndComp
 $Comp
 L Connector:Jack-DC J?
 U 1 1 607A5C33
-P 750 1000
+P 4100 6000
 AR Path="/608A4ECC/607A5C33" Ref="J?"  Part="1"
 AR Path="/607A5C33" Ref="J3"  Part="1"
-F 0 "J3" H 521 958 50  0000 R CNN
-F 1 "Jack-DC" H 521 1049 50  0000 R CNN
-F 2 "" H 800 960 50  0001 C CNN
-F 3 "~" H 800 960 50  0001 C CNN
-	1    750  1000
+F 0 "J3" H 4150 5800 50  0000 R CNN
+F 1 "Jack-DC" H 4250 5700 50  0000 R CNN
+F 2 "" H 4150 5960 50  0001 C CNN
+F 3 "~" H 4150 5960 50  0001 C CNN
+	1    4100 6000
 	1    0    0    1
 $EndComp
 Wire Wire Line
-	1050 1100 1200 1100
-Wire Wire Line
-	1200 1100 1200 1350
+	4400 5900 4500 5900
+$Comp
+L power:GND #PWR?
+U 1 1 60E32005
+P 4500 5900
+F 0 "#PWR?" H 4500 5650 50  0001 C CNN
+F 1 "GND" V 4505 5772 50  0000 R CNN
+F 2 "" H 4500 5900 50  0001 C CNN
+F 3 "" H 4500 5900 50  0001 C CNN
+	1    4500 5900
+	0    -1   -1   0
+$EndComp
+Wire Wire Line
+	4400 6100 4500 6100
+$Comp
+L power:+5V #PWR?
+U 1 1 60E39F6A
+P 4500 6100
+F 0 "#PWR?" H 4500 5950 50  0001 C CNN
+F 1 "+5V" V 4515 6228 50  0000 L CNN
+F 2 "" H 4500 6100 50  0001 C CNN
+F 3 "" H 4500 6100 50  0001 C CNN
+	1    4500 6100
+	0    1    1    0
+$EndComp
+Connection ~ 2700 4900
+$Comp
+L Kube_library:R R15
+U 1 1 6095BC8F
+P 2700 5100
+F 0 "R15" H 2700 5325 50  0000 C CNN
+F 1 "10K" H 2700 5234 50  0000 C CNN
+F 2 "" H 2700 5100 50  0001 C CNN
+F 3 "" H 2700 5100 50  0001 C CNN
+	1    2700 5100
+	0    -1   -1   0
+$EndComp
 $EndSCHEMATC

Commit message: footprints done
Parts:
- C1, C18, C2, C3, C4, C5, C6: footprint (none) -> Le_kube:C_0603_1608Metric_Pad1.08x0.95mm_HandSolder
- CP0: footprint (none) -> Le_kube:C_0603_1608Metric_Pad1.08x0.95mm_HandSolder; symbol Device:CP -> Le_kube-rescue:CP-Device
- J2: footprint (none) -> Le_kube:USB-A-TH_USB-302-T
- J3: footprint (none) -> Le_kube:PORT-JACK(DC-IN-TH_DC-003-2A-1.3)
- LDR1: footprint (none) -> Le_kube:LDR(RES-TH_L5.1-W4.3-P3.40-D0.5)
- Q1: footprint Package_TO_SOT_THT:TO-220-3_Vertical -> Le_kube:MOSFET(DPAK_L6.5-W6.0-P2.29-LS9.9-BR)
- R1, R15, R2, R3, R4, R5: footprint (none) -> Le_kube:R_0603_1608Metric_Pad0.98x0.95mm_HandSolder
- SW1: footprint (none) -> Le_kube:SW-TH_L8.0-W5.11-P5.08_TP11SH8CQE
- SW2, SW3, SW4, SW5: footprint (none) -> Le_kube:KEY-SMD_4P-L12.0-W12.0-P5.00-LS15.2
- U0: footprint Package_QFP:TQFP-32_7x7mm_P0.8mm -> Le_kube:ATMEGA328PB-AU(TQFP-32_L7.0-W7.0-P0.80-LS9.0-BL); symbol MCU_Microchip_ATmega:ATmega328PB-AU -> Le_kube-rescue:ATmega328PB-AU-MCU_Microchip_ATmega
- U4: footprint XCVR_ESP8266-01/ESP-01 -> Le_kube:ESP-01S(WIFIM-TH_8P-L24.7-W14.4-P2.54)
- VR1: footprint (none) -> Le_kube:LD1117(SOT-223_L6.7-W3.5-P2.30-BR)
- Y1: footprint (none) -> Le_kube:Crystal(HC-49S_L11.4-W4.8)
Changed lines of the file:
@@
 F 0 "R2" V 8250 3000 50  0000 L CNN
 F 1 "10K" V 8350 3000 50  0000 L CNN
-F 2 "" H 8450 3050 50  0001 C CNN
+F 2 "Le_kube:R_0603_1608Metric_Pad0.98x0.95mm_HandSolder" H 8450 3050 50  0001 C CNN
 F 3 "~" H 8450 3050 50  0001 C CNN
 	1    8450 3050
@@
 F 0 "R5" H 9859 3596 50  0000 L CNN
 F 1 "10K" H 9859 3505 50  0000 L CNN
-F 2 "" H 9800 3550 50  0001 C CNN
+F 2 "Le_kube:R_0603_1608Metric_Pad0.98x0.95mm_HandSolder" H 9800 3550 50  0001 C CNN
 F 3 "~" H 9800 3550 50  0001 C CNN
 	1    9800 3550
@@
 F 0 "SW5" H 10350 4035 50  0000 C CNN
 F 1 "SW_Push" H 10350 3944 50  0000 C CNN
-F 2 "" H 10350 3950 50  0001 C CNN
+F 2 "Le_kube:KEY-SMD_4P-L12.0-W12.0-P5.00-LS15.2" H 10350 3950 50  0001 C CNN
 F 3 "~" H 10350 3950 50  0001 C CNN
 	1    10350 3750
@@
 F 0 "R4" H 8409 3496 50  0000 L CNN
 F 1 "10K" H 8409 3405 50  0000 L CNN
-F 2 "" H 8350 3450 50  0001 C CNN
+F 2 "Le_kube:R_0603_1608Metric_Pad0.98x0.95mm_HandSolder" H 8350 3450 50  0001 C CNN
 F 3 "~" H 8350 3450 50  0001 C CNN
 	1    8350 3450
@@
 F 0 "SW4" H 8900 3935 50  0000 C CNN
 F 1 "SW_Push" H 8900 3844 50  0000 C CNN
-F 2 "" H 8900 3850 50  0001 C CNN
+F 2 "Le_kube:KEY-SMD_4P-L12.0-W12.0-P5.00-LS15.2" H 8900 3850 50  0001 C CNN
 F 3 "~" H 8900 3850 50  0001 C CNN
 	1    8900 3650
@@
 F 0 "R3" H 6909 3396 50  0000 L CNN
 F 1 "10K" H 6909 3305 50  0000 L CNN
-F 2 "" H 6850 3350 50  0001 C CNN
+F 2 "Le_kube:R_0603_1608Metric_Pad0.98x0.95mm_HandSolder" H 6850 3350 50  0001 C CNN
 F 3 "~" H 6850 3350 50  0001 C CNN
 	1    6850 3350
@@
 F 0 "SW3" H 7400 3835 50  0000 C CNN
 F 1 "SW_Push" H 7400 3744 50  0000 C CNN
-F 2 "" H 7400 3750 50  0001 C CNN
+F 2 "Le_kube:KEY-SMD_4P-L12.0-W12.0-P5.00-LS15.2" H 7400 3750 50  0001 C CNN
 F 3 "~" H 7400 3750 50  0001 C CNN
 	1    7400 3550
@@
 F 0 "R1" H 7209 2596 50  0000 L CNN
 F 1 "10K" H 7209 2505 50  0000 L CNN
-F 2 "" H 7150 2550 50  0001 C CNN
+F 2 "Le_kube:R_0603_1608Metric_Pad0.98x0.95mm_HandSolder" H 7150 2550 50  0001 C CNN
 F 3 "~" H 7150 2550 50  0001 C CNN
 	1    7150 2550
@@
 F 0 "LDR1" H 7567 3165 50  0000 C CNN
 F 1 "LDR" H 7567 3074 50  0000 C CNN
-F 2 "" H 7550 2750 50  0001 C CNN
+F 2 "Le_kube:LDR(RES-TH_L5.1-W4.3-P3.40-D0.5)" H 7550 2750 50  0001 C CNN
 F 3 "" H 7550 2750 50  0001 C CNN
 	1    7550 2750
@@
 F 0 "U4" H 9400 6467 50  0000 C CNN
 F 1 "ESP8266-01_ESP-01" H 9400 6376 50  0000 C CNN
-F 2 "XCVR_ESP8266-01/ESP-01" H 9400 5800 50  0001 L BNN
+F 2 "Le_kube:ESP-01S(WIFIM-TH_8P-L24.7-W14.4-P2.54)" H 9400 5800 50  0001 L BNN
 F 3 "" H 9400 5800 50  0001 L BNN
 F 4 "AI-Thinkers vendor" H 9400 5800 50  0001 L BNN "MANUFACTURER"
@@
 F 0 "C2" V 2654 1365 50  0000 L CNN
 F 1 "10µF" V 2745 1365 50  0000 L CNN
-F 2 "" V 2850 1288 50  0001 C CNN
+F 2 "Le_kube:C_0603_1608Metric_Pad1.08x0.95mm_HandSolder" V 2850 1288 50  0001 C CNN
 F 3 "~" H 2700 1250 50  0001 C CNN
 	1    2700 1250
@@
 F 0 "Q1" H 2005 2396 50  0000 L CNN
 F 1 "IRLB8721PBF" H 2005 2305 50  0000 L CNN
-F 2 "Package_TO_SOT_THT:TO-220-3_Vertical" H 2050 2275 50  0001 L CIN
+F 2 "Le_kube:MOSFET(DPAK_L6.5-W6.0-P2.29-LS9.9-BR)" H 2050 2275 50  0001 L CIN
 F 3 "http://www.infineon.com/dgdl/irlb8721pbf.pdf?fileId=5546d462533600a40153566056732591" H 1800 2350 50  0001 L CNN
 	1    1800 2350
@@
 F 0 "J2" H 1807 3767 50  0000 C CNN
 F 1 "USB_A" H 1807 3676 50  0000 C CNN
-F 2 "" H 1900 3250 50  0001 C CNN
+F 2 "Le_kube:USB-A-TH_USB-302-T" H 1900 3250 50  0001 C CNN
 F 3 " ~" H 1900 3250 50  0001 C CNN
 	1    1750 3300
@@
 F 0 "SW1" H 1250 1050 50  0000 C CNN
 F 1 "I/O" H 1250 1150 50  0000 C CNN
-F 2 "" H 1250 900 50  0001 C CNN
+F 2 "Le_kube:SW-TH_L8.0-W5.11-P5.08_TP11SH8CQE" H 1250 900 50  0001 C CNN
 F 3 "~" H 1250 900 50  0001 C CNN
 	1    1250 900
@@
 F 0 "VR1" H 2300 1100 50  0000 C CNN
 F 1 "LD1117" H 2300 1200 50  0000 C CNN
-F 2 "" H 2200 950 50  0001 C CNN
+F 2 "Le_kube:LD1117(SOT-223_L6.7-W3.5-P2.30-BR)" H 2200 950 50  0001 C CNN
 F 3 "" H 2200 950 50  0001 C CNN
 	1    2300 900
@@
 F 0 "C6" H 8392 2596 50  0000 L CNN
 F 1 "100nF" H 8392 2505 50  0000 L CNN
-F 2 "" H 8300 2550 50  0001 C CNN
+F 2 "Le_kube:C_0603_1608Metric_Pad1.08x0.95mm_HandSolder" H 8300 2550 50  0001 C CNN
 F 3 "~" H 8300 2550 50  0001 C CNN
 	1    8300 2550
@@
 	7150 2750 4500 2750
 $Comp
-L MCU_Microchip_ATmega:ATmega328PB-AU U0
+L Le_kube-rescue:ATmega328PB-AU-MCU_Microchip_ATmega U0
 U 1 1 6081701B
 P 3900 2750
 F 0 "U0" H 3850 2650 50  0000 C CNN
 F 1 "ATmega328PB-AU" H 3850 2900 50  0000 C CNN
-F 2 "Package_QFP:TQFP-32_7x7mm_P0.8mm" H 3900 2750 50  0001 C CIN
+F 2 "Le_kube:ATMEGA328PB-AU(TQFP-32_L7.0-W7.0-P0.80-LS9.0-BL)" H 3900 2750 50  0001 C CIN
 F 3 "http://ww1.microchip.com/downloads/en/DeviceDoc/40001906C.pdf" H 3900 2750 50  0001 C CNN
 	1    3900 2750
@@
 F 0 "SW2" H 6500 2550 50  0000 C CNN
 F 1 "RST" H 6500 2650 50  0000 C CNN
-F 2 "" H 6500 2550 50  0001 C CNN
+F 2 "Le_kube:KEY-SMD_4P-L12.0-W12.0-P5.00-LS15.2" H 6500 2550 50  0001 C CNN
 F 3 "~" H 6500 2550 50  0001 C CNN
 	1    6500 2350
@@
 F 0 "C4" V 5500 1950 50  0000 L CNN
 F 1 "34pF" V 5650 1900 50  0000 L CNN
-F 2 "" H 5850 2000 50  0001 C CNN
+F 2 "Le_kube:C_0603_1608Metric_Pad1.08x0.95mm_HandSolder" H 5850 2000 50  0001 C CNN
 F 3 "~" H 5850 2000 50  0001 C CNN
 	1    5850 2000
@@
 F 0 "C5" V 5950 2300 50  0000 C CNN
 F 1 "34pF" V 6050 2300 50  0000 C CNN
-F 2 "" H 5850 2300 50  0001 C CNN
+F 2 "Le_kube:C_0603_1608Metric_Pad1.08x0.95mm_HandSolder" H 5850 2300 50  0001 C CNN
 F 3 "~" H 5850 2300 50  0001 C CNN
 	1    5850 2300
@@
 F 0 "Y1" V 5304 2235 50  0000 L CNN
 F 1 "Crystal" V 5395 2235 50  0000 L CNN
-F 2 "" H 5350 2150 50  0001 C CNN
+F 2 "Le_kube:Crystal(HC-49S_L11.4-W4.8)" H 5350 2150 50  0001 C CNN
 F 3 "~" H 5350 2150 50  0001 C CNN
 	1    5350 2150
@@
 F 0 "C3" H 3200 1900 50  0000 L CNN
 F 1 "0.1µF" H 3150 1800 50  0000 L CNN
-F 2 "" H 3050 1850 50  0001 C CNN
+F 2 "Le_kube:C_0603_1608Metric_Pad1.08x0.95mm_HandSolder" H 3050 1850 50  0001 C CNN
 F 3 "~" H 3050 1850 50  0001 C CNN
 	1    3050 1850
@@
 F 0 "C18" V 5300 1250 50  0000 L CNN
 F 1 "100nF" V 5200 1200 50  0000 L CNN
-F 2 "" H 5450 1300 50  0001 C CNN
+F 2 "Le_kube:C_0603_1608Metric_Pad1.08x0.95mm_HandSolder" H 5450 1300 50  0001 C CNN
 F 3 "~" H 5450 1300 50  0001 C CNN
 	1    5450 1300
@@
 	5750 1150 5750 1000
 $Comp
-L Device:CP CP0
+L Le_kube-rescue:CP-Device CP0
 U 1 1 60D13B58
 P 5450 1000
 F 0 "CP0" V 5700 1000 50  0000 C CNN
 F 1 "10µF" V 5600 1000 50  0000 C CNN
-F 2 "" H 5488 850 50  0001 C CNN
+F 2 "Le_kube:C_0603_1608Metric_Pad1.08x0.95mm_HandSolder" H 5488 850 50  0001 C CNN
 F 3 "~" H 5450 1000 50  0001 C CNN
 	1    5450 1000
@@
 F 0 "C1" V 1946 1135 50  0000 R CNN
 F 1 "100nF" V 1855 1135 50  0000 R CNN
-F 2 "" V 2050 1288 50  0001 C CNN
+F 2 "Le_kube:C_0603_1608Metric_Pad1.08x0.95mm_HandSolder" V 2050 1288 50  0001 C CNN
 F 3 "~" H 1900 1250 50  0001 C CNN
 	1    1900 1250
@@
 F 0 "J3" H 4150 5800 50  0000 R CNN
 F 1 "Jack-DC" H 4250 5700 50  0000 R CNN
-F 2 "" H 4150 5960 50  0001 C CNN
+F 2 "Le_kube:PORT-JACK(DC-IN-TH_DC-003-2A-1.3)" H 4150 5960 50  0001 C CNN
 F 3 "~" H 4150 5960 50  0001 C CNN
 	1    4100 6000
@@
 	4400 5900 4500 5900
 $Comp
-L power:GND #PWR?
+L power:GND #PWR0147
 U 1 1 60E32005
 P 4500 5900
-F 0 "#PWR?" H 4500 5650 50  0001 C CNN
+F 0 "#PWR0147" H 4500 5650 50  0001 C CNN
 F 1 "GND" V 4505 5772 50  0000 R CNN
 F 2 "" H 4500 5900 50  0001 C CNN
@@
 	4400 6100 4500 6100
 $Comp
-L power:+5V #PWR?
+L power:+5V #PWR0148
 U 1 1 60E39F6A
 P 4500 6100
-F 0 "#PWR?" H 4500 5950 50  0001 C CNN
+F 0 "#PWR0148" H 4500 5950 50  0001 C CNN
 F 1 "+5V" V 4515 6228 50  0000 L CNN
 F 2 "" H 4500 6100 50  0001 C CNN
@@
 F 0 "R15" H 2700 5325 50  0000 C CNN
 F 1 "10K" H 2700 5234 50  0000 C CNN
-F 2 "" H 2700 5100 50  0001 C CNN
+F 2 "Le_kube:R_0603_1608Metric_Pad0.98x0.95mm_HandSolder" H 2700 5100 50  0001 C CNN
 F 3 "" H 2700 5100 50  0001 C CNN
 	1    2700 5100

Commit message: debut routage
Parts:
- removed J3: Jack-DC, Le_kube:PORT-JACK(DC-IN-TH_DC-003-2A-1.3), symbol Connector:Jack-DC
- added J3: Barrel_Jack_Switch, Le_kube:PORT-JACK(DC-IN-TH_DC-003-2A-1.3), symbol Kube_library:Barrel_Jack_Switch
- C3: value 0.1µF -> 100nF
- C4, C5: value 34pF -> 30pF
- Q1: symbol Transistor_FET:IRLB8721PBF -> Le_kube-rescue:IRLB8721PBF-Transistor_FET
Connections:
- wire segments 100 -> 103
Other:
- moved on the sheet: C1, C18, C2, C3, C4, C5, C6, CP0, J2, LDR1, R1, R15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

Commit message: routage done
Parts:
- SW2, SW3, SW4, SW5: symbol Switch:SW_Push -> Le_kube-rescue:SW_Push-Switch
- VR1: symbol Kube_library:LD1117 -> Le_kube-rescue:LD1117-Kube_library
Changed lines of the file:
@@
 $EndComp
 $Comp
-L Switch:SW_Push SW5
+L Le_kube-rescue:SW_Push-Switch SW5
 U 1 1 6073EFB3
 P 10550 3875
@@
 $EndComp
 $Comp
-L Switch:SW_Push SW4
+L Le_kube-rescue:SW_Push-Switch SW4
 U 1 1 60738C1C
 P 9100 3775
@@
 $EndComp
 $Comp
-L Switch:SW_Push SW3
+L Le_kube-rescue:SW_Push-Switch SW3
 U 1 1 607269BE
 P 7600 3675
@@
 $EndComp
 $Comp
-L Kube_library:LD1117 VR1
+L Le_kube-rescue:LD1117-Kube_library VR1
 U 1 1 60AB15B9
 P 2500 1025
@@
 $EndComp
 $Comp
-L Switch:SW_Push SW2
+L Le_kube-rescue:SW_Push-Switch SW2
 U 1 1 6075C822
 P 6700 2475

Commit message: routage done 4
Parts:
- SW2, SW3, SW4, SW5: symbol Le_kube-rescue:SW_Push-Switch -> Kube_library:SW
Connections:
- net +3V3: now also SW3.4, SW4.4, SW5.4; no longer SW3.2, SW4.2, SW5.2
- net GND: now also SW2.4; no longer SW2.2
Changed lines of the file:
@@
 $EndComp
 $Comp
-L Le_kube-rescue:SW_Push-Switch SW5
+L Kube_library:SW SW5
 U 1 1 6073EFB3
 P 10550 3875
@@
 $EndComp
 $Comp
-L Le_kube-rescue:SW_Push-Switch SW4
+L Kube_library:SW SW4
 U 1 1 60738C1C
 P 9100 3775
@@
 	7050 3575 7050 3675
 $Comp
-L Device:R_Small R3
-U 1 1 60734D6E
-P 7050 3475
-F 0 "R3" H 7109 3521 50  0000 L CNN
-F 1 "10K" H 7109 3430 50  0000 L CNN
-F 2 "Le_kube:R_0603_1608Metric_Pad0.98x0.95mm_HandSolder" H 7050 3475 50  0001 C CNN
-F 3 "~" H 7050 3475 50  0001 C CNN
-	1    7050 3475
-	1    0    0    -1
-$EndComp
-$Comp
 L power:+3.3V #PWR0107
 U 1 1 60733B39
@@
 $EndComp
 $Comp
-L Le_kube-rescue:SW_Push-Switch SW3
+L Kube_library:SW SW3
 U 1 1 607269BE
 P 7600 3675
@@
 $EndComp
 $Comp
-L Le_kube-rescue:SW_Push-Switch SW2
+L Kube_library:SW SW2
 U 1 1 6075C822
 P 6700 2475
@@
 	1    0    0    -1
 $EndComp
+$Comp
+L Device:R_Small R3
+U 1 1 60734D6E
+P 7050 3475
+F 0 "R3" H 7109 3521 50  0000 L CNN
+F 1 "10K" H 7109 3430 50  0000 L CNN
+F 2 "Le_kube:R_0603_1608Metric_Pad0.98x0.95mm_HandSolder" H 7050 3475 50  0001 C CNN
+F 3 "~" H 7050 3475 50  0001 C CNN
+	1    7050 3475
+	1    0    0    -1
+$EndComp
