File: Le_kube/ssd1306_128_64.sch (KiCad schematic (older format))
At the start: 2 parts

Commit message: continue on kicad_ssd1306
Parts:
- removed C1_screen: 0.1µF, symbol Kube_library:0.1µF
- removed UG-2864HSWEG01?: 128x64_OLED, symbol Kube_library:128x64_OLED
- added J?: J1, symbol Kube_library:J1
- added R1, R2, R3, R4: 4.7K, symbol Kube_library:R
- added R5: 910K, symbol Kube_library:R
- added U: 128x64_OLED, symbol Kube_library:128x64_OLED
Connections:
- net labels added: GND, VCC
- wire segments 0 -> 31
- no-connect marks 0 -> 1
Changed lines of the file:
@@
 $EndDescr
 $Comp
-L Kube_library:128x64_OLED UG-2864HSWEG01?
-U 1 1 60672303
-P 3750 3400
-F 0 "UG-2864HSWEG01?" H 3558 5015 50  0000 C CNN
-F 1 "128x64_OLED" H 3558 4924 50  0000 C CNN
-F 2 "" H 3750 3400 50  0001 C CNN
-F 3 "~" H 3750 3400 50  0001 C CNN
-	1    3750 3400
-	1    0    0    -1
-$EndComp
-$Comp
-L Kube_library:0.1µF C1_screen
-U 1 1 606744F1
-P 6750 2800
-F 0 "C1_screen" V 6704 2915 50  0000 L CNN
-F 1 "0.1µF" V 6795 2915 50  0000 L CNN
-F 2 "" V 6900 2838 50  0001 C CNN
-F 3 "~" H 6750 2800 50  0001 C CNN
-	1    6750 2800
-	0    1    1    0
+L Kube_library:128x64_OLED U
+U 1 1 606CAE59
+P 9000 2750
+F 0 "U" H 8500 1300 50  0000 C CNN
+F 1 "128x64_OLED" H 8500 1450 50  0000 C CNN
+F 2 "" H 9000 2750 50  0001 C CNN
+F 3 "~" H 9000 2750 50  0001 C CNN
+	1    9000 2750
+	1    0    0    -1
+$EndComp
+$Comp
+L Kube_library:R R1
+U 1 1 606D3DEF
+P 4200 1500
+F 0 "R1" V 4154 1588 50  0000 L CNN
+F 1 "4.7K" V 4245 1588 50  0000 L CNN
+F 2 "" H 4200 1500 50  0001 C CNN
+F 3 "" H 4200 1500 50  0001 C CNN
+	1    4200 1500
+	0    1    1    0
+$EndComp
+$Comp
+L Kube_library:R R2
+U 1 1 606D4491
+P 4550 1500
+F 0 "R2" V 4504 1588 50  0000 L CNN
+F 1 "4.7K" V 4595 1588 50  0000 L CNN
+F 2 "" H 4550 1500 50  0001 C CNN
+F 3 "" H 4550 1500 50  0001 C CNN
+	1    4550 1500
+	0    1    1    0
+$EndComp
+Wire Wire Line
+	4550 1300 4200 1300
+Connection ~ 4200 1300
+Wire Wire Line
+	4200 1300 3800 1300
+Text Label 3800 1300 0    50   ~ 0
+VCC
+$Comp
+L Kube_library:R R4
+U 1 1 606D4D1A
+P 4550 2400
+F 0 "R4" V 4504 2488 50  0000 L CNN
+F 1 "4.7K" V 4595 2488 50  0000 L CNN
+F 2 "" H 4550 2400 50  0001 C CNN
+F 3 "" H 4550 2400 50  0001 C CNN
+	1    4550 2400
+	0    1    1    0
+$EndComp
+$Comp
+L Kube_library:R R3
+U 1 1 606D54AA
+P 4200 2400
+F 0 "R3" V 4154 2488 50  0000 L CNN
+F 1 "4.7K" V 4245 2488 50  0000 L CNN
+F 2 "" H 4200 2400 50  0001 C CNN
+F 3 "" H 4200 2400 50  0001 C CNN
+	1    4200 2400
+	0    1    1    0
+$EndComp
+Wire Wire Line
+	4200 1700 4200 2050
+Wire Wire Line
+	4550 1700 4550 1950
+Wire Wire Line
+	6150 2050 4200 2050
+Connection ~ 4200 2050
+Wire Wire Line
+	4200 2050 4200 2200
+Wire Wire Line
+	6150 1950 4550 1950
+Connection ~ 4550 1950
+Wire Wire Line
+	4550 1950 4550 2200
+Wire Wire Line
+	4200 2600 4550 2600
+Wire Wire Line
+	4200 2600 4200 2800
+Connection ~ 4200 2600
+$Comp
+L power:GND #PWR?
+U 1 1 606D6329
+P 4200 2800
+F 0 "#PWR?" H 4200 2550 50  0001 C CNN
+F 1 "GND" H 4205 2627 50  0000 C CNN
+F 2 "" H 4200 2800 50  0001 C CNN
+F 3 "" H 4200 2800 50  0001 C CNN
+	1    4200 2800
+	1    0    0    -1
+$EndComp
+Wire Wire Line
+	7900 1900 7500 1900
+$Comp
+L power:GND #PWR?
+U 1 1 606D7059
+P 7500 1900
+F 0 "#PWR?" H 7500 1650 50  0001 C CNN
+F 1 "GND" V 7505 1772 50  0000 R CNN
+F 2 "" H 7500 1900 50  0001 C CNN
+F 3 "" H 7500 1900 50  0001 C CNN
+	1    7500 1900
+	0    1    1    0
+$EndComp
+$Comp
+L Kube_library:R R5
+U 1 1 606D72A6
+P 7350 2250
+F 0 "R5" H 7500 2350 50  0000 C CNN
+F 1 "910K" H 7200 2350 50  0000 C CNN
+F 2 "" H 7350 2250 50  0001 C CNN
+F 3 "" H 7350 2250 50  0001 C CNN
+	1    7350 2250
+	-1   0    0    1
+$EndComp
+Wire Wire Line
+	7550 2250 7850 2250
+Wire Wire Line
+	6700 2250 7150 2250
+$Comp
+L power:GND #PWR?
+U 1 1 606D94A8
+P 6700 2250
+F 0 "#PWR?" H 6700 2000 50  0001 C CNN
+F 1 "GND" V 6705 2122 50  0000 R CNN
+F 2 "" H 6700 2250 50  0001 C CNN
+F 3 "" H 6700 2250 50  0001 C CNN
+	1    6700 2250
+	0    1    1    0
+$EndComp
+Wire Wire Line
+	10150 1900 10500 1900
+Wire Wire Line
+	10500 1900 10500 2100
+Wire Wire Line
+	10150 2000 10350 2000
+NoConn ~ 10350 2000
+$Comp
+L power:GND #PWR?
+U 1 1 606DA2EF
+P 10500 2800
+F 0 "#PWR?" H 10500 2550 50  0001 C CNN
+F 1 "GND" H 10505 2627 50  0000 C CNN
+F 2 "" H 10500 2800 50  0001 C CNN
+F 3 "" H 10500 2800 50  0001 C CNN
+	1    10500 2800
+	1    0    0    -1
+$EndComp
+Wire Wire Line
+	10150 2100 10500 2100
+Connection ~ 10500 2100
+Wire Wire Line
+	10500 2100 10500 2200
+Wire Wire Line
+	10150 2200 10500 2200
+Connection ~ 10500 2200
+Wire Wire Line
+	10500 2200 10500 2300
+Wire Wire Line
+	10150 2300 10500 2300
+Connection ~ 10500 2300
+Wire Wire Line
+	10500 2300 10500 2400
+Wire Wire Line
+	10150 2400 10500 2400
+Connection ~ 10500 2400
+Wire Wire Line
+	10500 2400 10500 2500
+Wire Wire Line
+	10150 2500 10500 2500
+Connection ~ 10500 2500
+Wire Wire Line
+	10500 2500 10500 2600
+Wire Wire Line
+	10150 2600 10500 2600
+Connection ~ 10500 2600
+Wire Wire Line
+	10500 2600 10500 2700
+Wire Wire Line
+	10150 2700 10500 2700
+Connection ~ 10500 2700
+Wire Wire Line
+	10500 2700 10500 2800
+Wire Wire Line
+	10150 2800 10500 2800
+Connection ~ 10500 2800
+$Comp
+L Kube_library:J1 J?
+U 1 1 606E61CD
+P 5200 2850
+F 0 "J?" H 5232 3317 50  0000 C CNN
+F 1 "J1" H 5232 3226 50  0000 C CNN
+F 2 "" H 5150 2800 50  0001 C CNN
+F 3 "~" H 5150 2800 50  0001 C CNN
+	1    5200 2850
+	1    0    0    -1
 $EndComp
 $EndSCHEMATC
