File: Le_kube/_autosave-Le_kube.sch (KiCad schematic (older format))
At the start: 12 parts

Commit message: SWIMMING POULE
Connections:
- net Ecran/SDA_D1: now reaches U?.22 (PE3)
- net Capteur_humidite/AOUT: now reaches U?.25 (PC2)
- net Sheet60669016/CS renamed Ecran/CS
- net Sheet60669016/DC renamed Ecran/DC
- net Sheet60669016/RES renamed Ecran/RES
- net Sheet60669016/SCK_D0: no longer names the net of U?.17 (PB5)
- net Sheet60669016/SDA_D1: no longer names the net of U?.15 (PB3)
- net Sheet606BA941/SCL renamed Thermometre/SCL
- net Sheet606BA941/SDA renamed Thermometre/SDA
Changed lines of the file:
@@
 S 8100 2850 950  300
 U 606BA942
-F0 "Sheet606BA941" 50
+F0 "Thermometre" 50
 F1 "LM75A_Temp_Sensor.sch" 50
 F2 "SDA" I L 8100 2950 50
@@
 S 8100 3550 1000 600
 U 60669017
-F0 "Sheet60669016" 50
+F0 "Ecran" 50
 F1 "ssd1306_128_64.sch" 50
 F2 "CS" I L 8100 4050 50
@@
 	5850 1650 5850 3650
 Wire Wire Line
-	3600 1950 5700 1950
-Wire Wire Line
-	5700 1950 5700 3750
-Wire Wire Line
-	5700 3750 8100 3750
-Wire Wire Line
-	3600 2150 5550 2150
-Wire Wire Line
 	5550 2150 5550 3850
 Wire Wire Line
@@
 Connection ~ 4400 1250
 $Sheet
-S 9050 2200 850  400
+S 4650 2250 550  200
 U 608A4ECC
-F0 "Sheet608A4ECB" 50
+F0 "Capteur_humidite" 50
 F1 "Capasitive_sensor.sch" 50
+F2 "AOUT" I L 4650 2350 50
 $EndSheet
+Wire Wire Line
+	3900 2350 3900 2750
+Wire Wire Line
+	3900 2750 3600 2750
+Wire Wire Line
+	3900 2350 4650 2350
+Wire Wire Line
+	6700 3750 6700 5900
+Wire Wire Line
+	6700 5900 2400 5900
+Wire Wire Line
+	2400 5900 2400 3650
+Wire Wire Line
+	6700 3750 8100 3750
 $EndSCHEMATC
