File: Le_kube/_autosave-Le_kube.sch (KiCad schematic (older format))
At the start: 26 parts, among them J2 USB_A, Q1 IRLB8721PBF, SW1 I/O, SW2 RST, SW3 SW_Push, SW4 SW_Push, SW5 SW_Push, U0 ATmega328PB-AU, U4 ESP8266-01_ESP-01, Y1 Crystal

Commit message: modif atmega328pb
Parts:
- C3: value 0.1µF -> 100nF
Changed lines of the file:
@@
 	1700 900  1700 2150
-$Comp
-L Switch:SW_SPST SW1
-U 1 1 60AA65EA
-P 1250 900
-F 0 "SW1" H 1250 1050 50  0000 C CNN
-F 1 "I/O" H 1250 1150 50  0000 C CNN
-F 2 "" H 1250 900 50  0001 C CNN
-F 3 "~" H 1250 900 50  0001 C CNN
-	1    1250 900
-	1    0    0    -1
-$EndComp
 $Comp
 L Kube_library:LD1117 VR1
@@
 P 3050 1850
 F 0 "C3" H 3200 1900 50  0000 L CNN
-F 1 "0.1µF" H 3150 1800 50  0000 L CNN
+F 1 "100nF" H 3150 1800 50  0000 L CNN
 F 2 "" H 3050 1850 50  0001 C CNN
 F 3 "~" H 3050 1850 50  0001 C CNN
@@
 $EndComp
 $Comp
-L power:+5V #PWR?
+L power:+5V #PWR0114
 U 1 1 60DDA66B
 P 1050 900
-F 0 "#PWR?" H 1050 750 50  0001 C CNN
+F 0 "#PWR0114" H 1050 750 50  0001 C CNN
 F 1 "+5V" H 1065 1073 50  0000 C CNN
 F 2 "" H 1050 900 50  0001 C CNN
@@
 	0    -1   -1   0
 $EndComp
+$Comp
+L Switch:SW_SPST SW1
+U 1 1 60AA65EA
+P 1250 900
+F 0 "SW1" H 1250 1050 50  0000 C CNN
+F 1 "I/O" H 1250 1150 50  0000 C CNN
+F 2 "" H 1250 900 50  0001 C CNN
+F 3 "~" H 1250 900 50  0001 C CNN
+	1    1250 900
+	1    0    0    -1
+$EndComp
 $EndSCHEMATC
