File: Le_kube/Connector_ISP.sch (KiCad schematic (older format))
At the start: 1 part, among them J1 Conn_01x06_Male

Commit message: footprints done
Parts:
- J1: footprint (none) -> Le_kube:AVR-ISP(IDC-TH_6P-P2.54_C11214)
Changed lines of the file:
@@
 F 0 "J1" H 4383 3875 50  0000 C CNN
 F 1 "Conn_01x06_Male" H 4383 3784 50  0000 C CNN
-F 2 "" H 4400 3450 50  0001 C CNN
+F 2 "Le_kube:AVR-ISP(IDC-TH_6P-P2.54_C11214)" H 4400 3450 50  0001 C CNN
 F 3 "~" H 4400 3450 50  0001 C CNN
 	1    4400 3450
