File: Le_kube/LM75A_Temp_Sensor.sch (KiCad schematic (older format))
At the start: 4 parts

Commit message: sheet finish ?
Parts:
- gave numbers to parts that had none: 3
Changed lines of the file:
@@
 $Descr A4 11693 8268
 encoding utf-8
-Sheet 2 4
+Sheet 4 5
 Title ""
 Date ""
@@
 	5400 2900 5650 2900
 $Comp
-L Device:C_Small C?
+L Device:C_Small C7
 U 1 1 606C3724
 P 5750 2900
-F 0 "C?" V 5521 2900 50  0000 C CNN
+F 0 "C7" V 5521 2900 50  0000 C CNN
 F 1 "100nF" V 5612 2900 50  0000 C CNN
 F 2 "" H 5750 2900 50  0001 C CNN
@@
 	4700 3050 4700 3150
 $Comp
-L Device:R_Small R?
+L Device:R_Small R6
 U 1 1 606D09E7
 P 4700 3250
-F 0 "R?" H 4759 3296 50  0000 L CNN
+F 0 "R6" H 4759 3296 50  0000 L CNN
 F 1 "10K" H 4759 3205 50  0000 L CNN
 F 2 "" H 4700 3250 50  0001 C CNN
@@
 	4700 3550 4500 3550
 $Comp
-L Device:R_Small R?
+L Device:R_Small R7
 U 1 1 606D1923
 P 4700 3750
-F 0 "R?" H 4759 3796 50  0000 L CNN
+F 0 "R7" H 4759 3796 50  0000 L CNN
 F 1 "10K" H 4759 3705 50  0000 L CNN
 F 2 "" H 4700 3750 50  0001 C CNN

Commit message: fin de la schematic
Parts:
- gave numbers to parts that had none: 1
Changed lines of the file:
@@
 $EndDescr
 $Comp
-L Sensor_Temperature:LM75C U?
+L Sensor_Temperature:LM75C U1
 U 1 1 606BAF16
 P 5400 3550
-F 0 "U?" H 5250 4050 50  0000 C CNN
+F 0 "U1" H 5250 4050 50  0000 C CNN
 F 1 "LM75A" H 5600 4050 50  0000 C CNN
 F 2 "" H 5400 3550 50  0001 C CNN
@@
 	5800 3650 5900 3650
 $Comp
-L power:GND #PWR?
+L power:GND #PWR0131
 U 1 1 606BC5F4
 P 5900 3650
-F 0 "#PWR?" H 5900 3400 50  0001 C CNN
+F 0 "#PWR0131" H 5900 3400 50  0001 C CNN
 F 1 "GND" H 5905 3477 50  0000 C CNN
 F 2 "" H 5900 3650 50  0001 C CNN
@@
 Connection ~ 5900 3650
 $Comp
-L power:GND #PWR?
+L power:GND #PWR0132
 U 1 1 606C179D
 P 5400 4050
-F 0 "#PWR?" H 5400 3800 50  0001 C CNN
+F 0 "#PWR0132" H 5400 3800 50  0001 C CNN
 F 1 "GND" H 5405 3877 50  0000 C CNN
 F 2 "" H 5400 4050 50  0001 C CNN
@@
 	5900 2900 5900 3000
 $Comp
-L power:GND #PWR?
+L power:GND #PWR0133
 U 1 1 606C5255
 P 5900 3000
-F 0 "#PWR?" H 5900 2750 50  0001 C CNN
+F 0 "#PWR0133" H 5900 2750 50  0001 C CNN
 F 1 "GND" H 5905 2827 50  0000 C CNN
 F 2 "" H 5900 3000 50  0001 C CNN
@@
 SCL
 $Comp
-L power:+3.3V #PWR?
+L power:+3.3V #PWR0134
 U 1 1 606CC412
 P 5400 2750
-F 0 "#PWR?" H 5400 2600 50  0001 C CNN
+F 0 "#PWR0134" H 5400 2600 50  0001 C CNN
 F 1 "+3.3V" H 5415 2923 50  0000 C CNN
 F 2 "" H 5400 2750 50  0001 C CNN
@@
 	4700 3850 4700 4000
 $Comp
-L power:+3.3V #PWR?
+L power:+3.3V #PWR0135
 U 1 1 606D255B
 P 4700 4000
-F 0 "#PWR?" H 4700 3850 50  0001 C CNN
+F 0 "#PWR0135" H 4700 3850 50  0001 C CNN
 F 1 "+3.3V" H 4715 4173 50  0000 C CNN
 F 2 "" H 4700 4000 50  0001 C CNN
@@
 Connection ~ 5400 2900
 $Comp
-L power:+3.3V #PWR?
+L power:+3.3V #PWR0136
 U 1 1 606D3BE0
 P 4700 3050
-F 0 "#PWR?" H 4700 2900 50  0001 C CNN
+F 0 "#PWR0136" H 4700 2900 50  0001 C CNN
 F 1 "+3.3V" H 4715 3223 50  0000 C CNN
 F 2 "" H 4700 3050 50  0001 C CNN

Commit message: footprints done
Parts:
- C7: footprint (none) -> Le_kube:C_0603_1608Metric_Pad1.08x0.95mm_HandSolder
- R6, R7: footprint (none) -> Le_kube:R_0603_1608Metric_Pad0.98x0.95mm_HandSolder
- U1: footprint (none) -> Le_kube:TEMP_SENSOR(SOIC-8_L5.0-W4.0-P1.27-LS6.0-BL)
Changed lines of the file:
@@
 F 0 "U1" H 5250 4050 50  0000 C CNN
 F 1 "LM75A" H 5600 4050 50  0000 C CNN
-F 2 "" H 5400 3550 50  0001 C CNN
+F 2 "Le_kube:TEMP_SENSOR(SOIC-8_L5.0-W4.0-P1.27-LS6.0-BL)" H 5400 3550 50  0001 C CNN
 F 3 "http://www.ti.com/lit/ds/symlink/lm75b.pdf" H 5400 3550 50  0001 C CNN
 	1    5400 3550
@@
 F 0 "C7" V 5521 2900 50  0000 C CNN
 F 1 "100nF" V 5612 2900 50  0000 C CNN
-F 2 "" H 5750 2900 50  0001 C CNN
+F 2 "Le_kube:C_0603_1608Metric_Pad1.08x0.95mm_HandSolder" H 5750 2900 50  0001 C CNN
 F 3 "~" H 5750 2900 50  0001 C CNN
 	1    5750 2900
@@
 F 0 "R6" H 4759 3296 50  0000 L CNN
 F 1 "10K" H 4759 3205 50  0000 L CNN
-F 2 "" H 4700 3250 50  0001 C CNN
+F 2 "Le_kube:R_0603_1608Metric_Pad0.98x0.95mm_HandSolder" H 4700 3250 50  0001 C CNN
 F 3 "~" H 4700 3250 50  0001 C CNN
 	1    4700 3250
@@
 F 0 "R7" H 4759 3796 50  0000 L CNN
 F 1 "10K" H 4759 3705 50  0000 L CNN
-F 2 "" H 4700 3750 50  0001 C CNN
+F 2 "Le_kube:R_0603_1608Metric_Pad0.98x0.95mm_HandSolder" H 4700 3750 50  0001 C CNN
 F 3 "~" H 4700 3750 50  0001 C CNN
 	1    4700 3750
