File: Le_kube/Le_kube.kicad_pcb (KiCad board)
At the start: 2 copper layers, 53 parts, among them J1 Conn_01x06_Male, J2 USB_A, J3 Barrel_Jack_Switch, Q1 IRLB8721PBF, SW1 I/O, SW2 RST, SW3 SW_Push, SW4 SW_Push, SW5 SW_Push, U0 ATmega328PB-AU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

Commit message: Routage
Parts:
- C19: footprint Le_kube:C_0603_1608Metric_Pad1.08x0.95mm_HandSolder -> Le_kube:PROBE
- moved R5 136.7 mm to (185.4, 46.8)
- moved C19 114.8 mm to (110.0, 112.0)
- moved R4 111.6 mm to (166.4, 46.1)
- moved C17 108.3 mm to (110.8, 105.8), turned to 90 degrees
- moved R12 107.8 mm to (109.1, 105.9), turned to 90 degrees
- moved D1 106.8 mm to (104.2, 104.9), turned to 180 degrees
- moved SW2 106.2 mm to (51.3, 111.9)
- moved R13 105.1 mm to (108.0, 102.6)
- moved U3 103.3 mm to (101.6, 98.7), turned to 90 degrees
- moved R11 101.8 mm to (100.8, 105.1), turned to 90 degrees
- moved C15 95.1 mm to (98.5, 105.3), turned to 90 degrees
- moved R14 94.8 mm to (96.3, 105.1), turned to 270 degrees
- moved R15 91.9 mm to (18.2, 87.1)
- moved C14 91.4 mm to (94.1, 105.0), turned to 90 degrees
- moved C16 89.7 mm to (95.6, 100.8), turned to 270 degrees
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Routing:
- net Net-(C19-Pad2): track 0.00 -> 155.1 mm
- net GND: track 0.00 -> 62.6 mm
- net Net-(C16-Pad1): track 0.00 -> 6.83 mm
- net Net-(R13-Pad2): track 0.00 -> 6.74 mm
- net /HUM: track 0.00 -> 5.43 mm

Commit message: routage en cours
Parts:
- removed R3, R4, R5: 10K, Le_kube:R_0603_1608Metric_Pad0.98x0.95mm_HandSolder
- C19, SW2, SW3, SW4, SW5: moved to B.Cu
- moved SW5 100.1 mm to (88.1, 89.1), turned to 90 degrees
- moved R15 75.1 mm to (92.7, 77.7)
- moved SW4 70.9 mm to (100.4, 89.1), turned to 90 degrees
- moved Q1 69.5 mm to (86.5, 88.2)
- moved J1 60.0 mm to (111.2, 74.0), turned to 270 degrees
- moved R2 57.8 mm to (107.8, 91.8)
- moved C6 51.4 mm to (107.8, 93.2), turned to 180 degrees
- moved J2 50.0 mm to (90.0, 101.8)
- moved SW2 49.7 mm to (100.2, 103.0), turned to 180 degrees
- moved U1 48.3 mm to (96.5, 99.8), turned to 180 degrees
- moved J3 47.0 mm to (85.2, 80.2)
- moved SW3 44.8 mm to (112.8, 89.1), turned to 90 degrees
- moved C1 35.7 mm to (89.7, 66.0), turned to 270 degrees
- moved R1 35.5 mm to (92.8, 72.0)
- moved VR1 35.0 mm to (80.9, 64.3)
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Routing:
- net +3V3: track 0.00 -> 160.8 mm, vias 0 -> 1
- net Net-(C19-Pad2): track 155.1 -> 4.23 mm
- net GND: track 62.6 -> 6.33 mm, vias 0 -> 3
- net Net-(R5-Pad2): track 0.00 -> 42.2 mm, vias 0 -> 1
- net /SCREEN_MISO: track 0.00 -> 37.3 mm, vias 0 -> 2
- net Net-(C1-Pad2): track 0.00 -> 36.3 mm
- net /HUM: track 5.43 -> 39.1 mm, vias 0 -> 2
- net /SCREEN_SCK: track 0.00 -> 32.6 mm, vias 0 -> 2
- net /SDA: track 0.00 -> 32.4 mm, vias 0 -> 2
- net /SCL: track 0.00 -> 30.9 mm, vias 0 -> 2
- net Net-(C15-Pad2): track 0.00 -> 28.2 mm, vias 0 -> 2
- net /SCREEN_SS: track 0.00 -> 26.1 mm, vias 0 -> 2
- net /ESP_TX: track 0.00 -> 25.6 mm, vias 0 -> 2
- net /SCREEN_MOSI: track 0.00 -> 25.0 mm, vias 0 -> 2
- net Net-(C6-Pad2): track 0.00 -> 24.7 mm, vias 0 -> 2
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Other:
- board outline added: 52 x 125 mm
- net class 5V added: clearance 0.2, trace_width 0.4, via_dia 0.8, via_drill 0.4
- net class Power added: clearance 0.2, trace_width 0.4, via_dia 0.8, via_drill 0.4

Commit message: debut du routage (commit de secours)
Parts:
- moved SW2 55.3 mm to (151.4, 82.0)
- moved Q1 5.49 mm to (81.0, 88.6)
- moved C8 5.11 mm to (91.8, 68.5), turned to 270 degrees
- moved J2 3.92 mm to (86.6, 99.8)
- moved C9 3.09 mm to (93.8, 68.5), turned to 270 degrees
- moved CP0 2.63 mm to (82.8, 71.6)
- moved C7 2.48 mm to (84.9, 80.5)
- moved J3 2.40 mm to (83.1, 81.3)
- moved C1 2.35 mm to (87.4, 66.5)
- moved C18 2.35 mm to (82.8, 69.8)
- moved C2 2.35 mm to (84.8, 66.5)
- moved VR1 2.35 mm to (78.6, 64.8)
- moved SW1 1.54 mm to (82.0, 74.9)
- moved C12 0.91 mm to (96.6, 68.3)
- moved Y1 0.85 mm to (99.6, 86.6)
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Routing:
- net +3V3: track 160.8 -> 35.4 mm, vias 1 -> 0
- net Net-(R5-Pad2): track 42.2 -> 0.00 mm, vias 1 -> 0
- net /SCREEN_MISO: track 37.3 -> 0.00 mm, vias 2 -> 0
- net /SCREEN_SCK: track 32.6 -> 0.00 mm, vias 2 -> 0
- net Net-(C1-Pad2): track 36.3 -> 7.81 mm
- net /SDA: track 32.4 -> 3.98 mm, vias 2 -> 0
- net /SCL: track 30.9 -> 3.07 mm, vias 2 -> 0
- net /HUM: track 39.1 -> 12.7 mm, vias 2 -> 0
- net /SCREEN_SS: track 26.1 -> 0.00 mm, vias 2 -> 0
- net /ESP_TX: track 25.6 -> 0.00 mm, vias 2 -> 0
- net /SCREEN_MOSI: track 25.0 -> 0.00 mm, vias 2 -> 0
- net Net-(C6-Pad2): track 24.7 -> 0.00 mm, vias 2 -> 0
- net /SCREEN_RST: track 22.4 -> 0.00 mm, vias 2 -> 0
- net Net-(Q1-Pad1): track 20.9 -> 0.00 mm
- net Net-(C4-Pad2): track 15.5 -> 0.00 mm, vias 2 -> 0
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
Commit message: conflit ?
Parts:
- moved SW2 55.3 mm to (100.2, 103.0)
- moved LDR1 26.3 mm to (92.9, 68.6)
- moved Q1 5.49 mm to (86.5, 88.2)
- moved C8 5.11 mm to (92.5, 63.4), turned to 0 degrees
- moved J2 3.92 mm to (90.0, 101.8)
- moved C9 3.09 mm to (94.5, 65.5), turned to 0 degrees
- moved CP0 2.63 mm to (81.3, 69.4)
- moved C7 2.48 mm to (87.4, 80.7)
- moved J3 2.40 mm to (85.2, 80.2)
- moved C1 2.35 mm to (89.7, 66.0)
- moved C18 2.35 mm to (85.1, 69.3)
- moved C2 2.35 mm to (87.1, 66.0)
- moved VR1 2.35 mm to (80.9, 64.3)
- moved SW1 1.54 mm to (82.6, 73.5)
- moved C12 0.91 mm to (97.5, 68.3)
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Routing:
- net +3V3: track 35.4 -> 167.0 mm, vias 0 -> 1
- net Net-(R5-Pad2): track 0.00 -> 42.1 mm, vias 0 -> 1
- net /SCREEN_MISO: track 0.00 -> 37.3 mm, vias 0 -> 2
- net Net-(C6-Pad2): track 0.00 -> 34.5 mm, vias 0 -> 3
- net /SCREEN_SCK: track 0.00 -> 32.6 mm, vias 0 -> 2
- net Net-(C1-Pad2): track 7.81 -> 36.3 mm
- net /SDA: track 3.98 -> 32.4 mm, vias 0 -> 2
- net Net-(R3-Pad2): track 0.00 -> 28.1 mm, vias 0 -> 1
- net /SCL: track 3.07 -> 30.9 mm, vias 0 -> 2
- net /HUM: track 12.7 -> 39.1 mm, vias 0 -> 2
- net /SCREEN_SS: track 0.00 -> 26.1 mm, vias 0 -> 2
- net /SCREEN_MOSI: track 0.00 -> 25.0 mm, vias 0 -> 2
- net /ESP_TX: track 0.00 -> 24.0 mm, vias 0 -> 2
- net /SCREEN_RST: track 0.00 -> 22.4 mm, vias 0 -> 2
- net Net-(Q1-Pad1): track 0.00 -> 20.9 mm
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
Commit message: routage done
Parts:
- moved U4 9.64 mm to (120.9, 82.3)
- moved J2 3.78 mm to (87.0, 99.5)
- moved J3 1.81 mm to (83.4, 80.0)
Routing:
- net GND: track 6.33 -> 251.6 mm, vias 3 -> 24
- net Net-(C19-Pad2): track 4.23 -> 64.7 mm, vias 0 -> 1
- net +3V3: track 167.0 -> 217.0 mm, vias 1 -> 4
- net /connecteur_isp/RST: track 0.00 -> 26.3 mm, vias 0 -> 2
- net /ISP_SCK: track 0.00 -> 18.8 mm
- net Net-(C1-Pad2): track 36.3 -> 54.5 mm, vias 0 -> 1
- net Net-(R4-Pad2): track 0.00 -> 16.4 mm, vias 0 -> 1
- net /ESP_RX: track 15.2 -> 29.8 mm
- net Net-(C5-Pad2): track 0.00 -> 10.8 mm, vias 0 -> 2
- net /ESP_TX: track 24.0 -> 34.0 mm
- net Net-(J2-Pad1): track 13.6 -> 12.1 mm
- net Net-(C15-Pad2): track 28.2 -> 29.2 mm
- net /SDA: track 32.4 -> 33.3 mm
- net /HUM: track 39.1 -> 38.2 mm
- net +5V: track 10.8 -> 10.0 mm
- added copper zone on B.Cu, net GND
Other:
- board size 52 x 125 mm -> 50 x 125 mm

Commit message: routage update
Parts:
- R1, SW1: moved to B.Cu
- moved U4 42.1 mm to (78.8, 82.0), turned to 0 degrees
- moved Q1 40.7 mm to (119.2, 64.0)
- moved J2 37.8 mm to (116.8, 76.2), turned to 90 degrees
- moved R15 33.4 mm to (123.0, 63.8)
- moved SW3 24.8 mm to (88.0, 89.1), turned to 270 degrees
- moved SW5 24.7 mm to (112.8, 89.1), turned to 270 degrees
- moved C7 19.6 mm to (93.0, 99.5)
- moved R6 18.6 mm to (98.0, 91.8), turned to 180 degrees
- moved R7 18.1 mm to (98.0, 93.2), turned to 0 degrees
- moved J1 17.8 mm to (120.0, 58.5), turned to 180 degrees
- moved C13 16.4 mm to (86.8, 57.5), turned to 90 degrees
- moved LDR1 15.3 mm to (78.0, 65.0), turned to 90 degrees
- moved SW1 15.0 mm to (77.7, 59.3), turned to 90 degrees
- moved R1 14.4 mm to (78.5, 73.8)
- moved C12 14.2 mm to (88.2, 57.5), turned to 90 degrees
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Connections:
- SW2 pad 2: GND -> (no net)
- SW2 pad 4: (no net) -> GND
- SW3 pad 2: +3V3 -> (no net)
- SW3 pad 4: (no net) -> +3V3
- SW4 pad 2: +3V3 -> (no net)
- SW4 pad 4: (no net) -> +3V3
- SW5 pad 2: +3V3 -> (no net)
- SW5 pad 4: (no net) -> +3V3
Routing:
- net GND: track 251.6 -> 143.1 mm, vias 24 -> 23
- net Net-(R5-Pad2): track 42.1 -> 5.97 mm
- net +3V3: track 217.0 -> 248.3 mm, vias 4 -> 6
- net Net-(Q1-Pad1): track 20.9 -> 42.5 mm, vias 0 -> 2
- net Net-(LDR1-Pad1): track 8.84 -> 27.6 mm, vias 0 -> 3
- net /ISP_MISO: track 9.71 -> 27.7 mm, vias 0 -> 1
- net /SCREEN_MISO: track 36.9 -> 19.7 mm, vias 2 -> 0
- net /ISP_MOSI: track 8.91 -> 25.6 mm
- net Net-(R3-Pad2): track 28.1 -> 12.6 mm
- net /SCREEN_SCK: track 32.6 -> 17.6 mm, vias 2 -> 0
- net Net-(C6-Pad2): track 34.5 -> 48.5 mm, vias 3 -> 5
- net /ESP_TX: track 34.0 -> 20.1 mm, vias 2 -> 0
- net Net-(R4-Pad2): track 16.4 -> 2.82 mm
- net /ISP_SCK: track 18.8 -> 29.5 mm
- net /ESP_RX: track 29.8 -> 19.4 mm
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Other:
- outline, holes or cut-outs redrawn

Commit message: routage done
Parts:
- removed SW1: I/O, Le_kube:SW-TH_L8.0-W5.11-P5.08_TP11SH8CQE
- added I O: I/O, Le_kube:SW-TH_L8.0-W5.11-P5.08_TP11SH8CQE, F.Cu at (78.3, 72.5)
- added R3: 10K, Le_kube:R_0603_1608Metric_Pad0.98x0.95mm_HandSolder, F.Cu at (90.5, 72.7)
- added R4: 10K, Le_kube:R_0603_1608Metric_Pad0.98x0.95mm_HandSolder, F.Cu at (90.5, 75.2)
- added R5: 10K, Le_kube:R_0603_1608Metric_Pad0.98x0.95mm_HandSolder, F.Cu at (94.9, 72.7)
- C19: value PROBE -> GROUND
- LDR1: moved to B.Cu
- R1: moved to F.Cu
- moved R1 13.2 mm to (76.6, 60.7), turned to 90 degrees
- moved J3 10.2 mm to (83.4, 80.0)
- moved U4 8.66 mm to (78.2, 90.6)
- moved LDR1 7.46 mm to (79.5, 57.7), turned to 270 degrees
- moved C19 6.70 mm to (100.5, 117.2)
- moved VR1 5.37 mm to (80.1, 64.7)
- moved C1 3.59 mm to (85.3, 64.2)
- moved C18 3.59 mm to (88.3, 64.2)
- moved CP0 3.59 mm to (86.8, 64.2)
- moved J2 0.54 mm to (116.8, 75.6)
- moved C2 0.17 mm to (87.2, 60.9)
Connections:
- J3 pad 1: +5V -> GND
- J3 pad 2: GND -> +5V
- SW2 pad 2: (no net) -> GND
- SW2 pad 4: GND -> (no net)
- SW3 pad 2: (no net) -> +3V3
- SW3 pad 4: +3V3 -> (no net)
- SW4 pad 2: (no net) -> +3V3
- SW4 pad 4: +3V3 -> (no net)
- SW5 pad 2: (no net) -> +3V3
- SW5 pad 4: +3V3 -> (no net)
Routing:
- net Net-(C19-Pad2): track 64.4 -> 40.0 mm
- net +3V3: track 248.3 -> 258.9 mm
- net Net-(LDR1-Pad1): track 27.6 -> 35.6 mm, vias 3 -> 2
- net /ESP_RX: track 19.4 -> 25.6 mm
- net Net-(C1-Pad2): track 55.4 -> 61.5 mm
- net +5V: track 12.4 -> 8.22 mm
- net /ESP_TX: track 20.1 -> 22.5 mm
- net GND: track 143.1 -> 142.9 mm, vias 23 -> 25
Other:
- board size 50 x 125 mm -> 51 x 133.1 mm
- rule trace_min: 0.2 -> 0.127
- rule via_min_drill: 0.3 -> 0.2
- board text added: "DWN"
- board text added: "Le_Kube"
- board text added: "RST"
- board text added: "SLCT"
- board text added: "UP"

Commit message: routage done 2
Parts:
- added G***: LOGO, Le_kube:logo, B.Cu at (89.1, 109.9)
- added G***: LOGO, Le_kube:logo, B.Cu at (111.4, 110.0)
Routing:
- net Net-(C19-Pad2): track 40.0 -> 39.4 mm
