File: Le_kube/Le_kube.kicad_pcb (KiCad board)
At the start: 2 copper layers, 51 x 133.1 mm, 55 parts, among them J1 Conn_01x06_Male, J2 USB_A, J3 Barrel_Jack_Switch, Q1 IRLB8721PBF, SW2 RST, SW3 SW_Push, SW4 SW_Push, SW5 SW_Push, U0 ATmega328PB-AU, U1 LM75A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

Commit message: routage done 3
Routing:
- net Net-(R4-Pad2): track 2.82 -> 3.64 mm

Commit message: routage done 4
Parts:
- C19: value GROUND -> PROBE
- SW1: renamed from I O
- moved R5 16.1 mm to (109.3, 79.8), turned to 180 degrees
- moved R3 7.31 mm to (85.5, 78.0), turned to 270 degrees
- moved R4 6.59 mm to (93.2, 81.3)
Connections:
- SW2 pad 2: GND -> (no net)
- SW2 pad 4: (no net) -> GND
- SW3 pad 2: +3V3 -> (no net)
- SW3 pad 4: (no net) -> +3V3
- SW4 pad 2: +3V3 -> (no net)
- SW4 pad 4: (no net) -> +3V3
- SW5 pad 2: +3V3 -> (no net)
- SW5 pad 4: (no net) -> +3V3
Routing:
- net GND: track 143.3 -> 150.3 mm, vias 25 -> 27
- net Net-(R4-Pad2): track 3.64 -> 7.70 mm
- net Net-(R3-Pad2): track 12.6 -> 15.6 mm, vias 1 -> 2
- net Net-(R5-Pad2): track 5.97 -> 8.03 mm
Other:
- board size 51 x 133.1 mm -> 51.6 x 133.4 mm
